File: KiCAD/StepperClock.kicad_sch (KiCad schematic)
At the start: 17 parts, among them J1 Screw_Terminal_01x02, J2 Conn_DCF77, J3 Conn_Hour_Home, J4 Conn_DCF77, J5 Conn_02x07_Odd_Even, J6 Conn_RGB_LED, J7 Conn__Motor_Hour, J8 Conn_Motor_Minute, U1 LM7805_TO220, U2 ULN2003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

Commit message: Long overdue updates
Other:
- title: (none) -> Main PCB
Changed lines of the file:
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@@
 (kicad_sch (version 20230121) (generator eeschema)
   (paper "A4")
+  (title_block
+    (title "Main PCB")
+    (date "2023-09-21")
+  )
   (junction (at 107.95 72.39) (diameter 0) (color 0 0 0 0)
   )
